File: kiCAD/schmatic/schmatic.kicad_pcb (KiCad board)
At the start: 2 copper layers, 38 parts, among them J2 Conn_02x03_Counter_Clockwise, J3 Connector, USB-TYPE-C-16P, U1 AMS1117, U2 MS561101BA03-50, U4 MPU-9250, U6 STM32F103C8T6, X1 X322516MLB4SI, X2 Q13FC1350000400

Commit message: feat: new PCB design and improved rocket flight sim
Parts:
- removed C6: 4.7uF, PCM_JLCPCB:C_0603
- added H1: MountingHole, MountingHole:MountingHole_2.2mm_M2_Pad, F.Cu at (129.5, 85.5)
- added H2: MountingHole, MountingHole:MountingHole_2.2mm_M2_Pad, F.Cu at (156.0, 85.5)
- added H3: MountingHole, MountingHole:MountingHole_2.2mm_M2_Pad, F.Cu at (129.5, 113.0)
- added H4: MountingHole, MountingHole:MountingHole_2.2mm_M2_Pad, F.Cu at (156.0, 113.0)
- added R3: 10kΩ, PCM_JLCPCB:R_0603, F.Cu at (150.2, 94.8)
- added R7: 10kΩ, PCM_JLCPCB:R_0603, F.Cu at (152.0, 94.8)
- moved X2 147.2 mm to (148.0, 85.0), turned to 90 degrees
- moved C3 146.0 mm to (147.8, 88.3)
- moved C2 144.0 mm to (147.8, 89.8)
- moved C5 142.6 mm to (147.2, 98.3)
- moved X1 142.2 mm to (138.2, 84.8), turned to -90 degrees
- moved L2 139.7 mm to (132.2, 90.3)
- moved J2 136.2 mm to (156.0, 102.6)
- moved U2 135.9 mm to (155.2, 93.3), turned to 90 degrees
- moved L1 134.5 mm to (138.7, 102.6), turned to 90 degrees
- moved C8 133.5 mm to (145.5, 84.0), turned to -90 degrees
- moved C12 133.4 mm to (141.5, 84.8), turned to 90 degrees
- moved C4 132.6 mm to (136.8, 98.3), turned to 180 degrees
- moved C7 131.2 mm to (145.5, 86.0), turned to 90 degrees
- moved C14 129.9 mm to (149.8, 91.8), turned to 90 degrees
- moved C11 127.9 mm to (135.8, 84.8), turned to -90 degrees
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Connections:
- R1 pad 2: /SDA -> /MPU_SDA
- R2 pad 2: /SCL -> /MPU_SCL
- U2 pad 7: /SDA -> /P_SDA
- U2 pad 8: /SCL -> /P_SCL
- U4 pad 23: /SCL -> /MPU_SCL
- U4 pad 24: /SDA -> /MPU_SDA
- U6 pad 21: unconnected-(U6-PB10-Pad21) -> /MPU_SCL
- U6 pad 22: unconnected-(U6-PB11-Pad22) -> /MPU_SDA
- U6 pad 42: unconnected-(U6-PB6-Pad42) -> /P_SCL
- U6 pad 43: unconnected-(U6-PB7-Pad43) -> /P_SDA
- U6 pad 45: /SCL -> unconnected-(U6-PB8-Pad45)
- U6 pad 46: /SDA -> unconnected-(U6-PB9-Pad46)
Routing:
- net +3.3VP: track 11.1 -> 126.7 mm, vias 0 -> 2
- net GND: track 25.9 -> 122.3 mm, vias 0 -> 23
- net /NRST: track 0.00 -> 24.8 mm, vias 0 -> 2
- net /SWO: track 0.00 -> 23.6 mm, vias 0 -> 1
- net /Boot0: track 0.00 -> 21.9 mm, vias 0 -> 2
- net /INT: track 0.00 -> 18.8 mm, vias 0 -> 2
- net +5V: track 0.00 -> 18.4 mm, vias 0 -> 2
- net /SWDIO: track 0.00 -> 15.5 mm
- net /SWCLK: track 0.00 -> 15.1 mm, vias 0 -> 1
- net /HSE_IN: track 0.00 -> 13.7 mm
- net Net-(J3-VBUS-PadA9B4): track 0.00 -> 12.7 mm
- net Net-(J3-CC1): track 0.00 -> 11.0 mm
- net /LSE_OUT: track 0.00 -> 9.90 mm
- net +3.3VA: track 0.00 -> 9.82 mm
- net Net-(J3-CC2): track 0.00 -> 8.42 mm
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- added copper zone on B.Cu, net GND
Other:
- board outline added: 33.5 x 34.5 mm
