File: kiCAD/schmatic/schmatic.kicad_sch (KiCad schematic)
At the start: 43 parts, among them J2 Conn_02x03_Counter_Clockwise, J3 Connector, USB-TYPE-C-16P, U1 AMS1117, U2 MS561101BA03-50, U4 MPU-9250, U6 STM32F103C8T6, X1 X322516MLB4SI, X2 Q13FC1350000400

Commit message: feat: modified PCB flight computer for extended features
Parts:
- removed C15: 100nF, PCM_JLCPCB:C_0402, symbol PCM_JLCPCB-Capacitors:0402,100nF
- removed J2: Conn_02x03_Counter_Clockwise, Connector_PinHeader_1.27mm:PinHeader_2x03_P1.27mm_Vertical, symbol Connector_Generic:Conn_02x03_Counter_Clockwise
- removed R6: 5.1kΩ, PCM_JLCPCB:R_0805, symbol PCM_JLCPCB-Resistors:0805,5.1kΩ
- added C15, C26, C27, C6: 10uF, PCM_JLCPCB:C_0603, symbol PCM_JLCPCB-Capacitors:0603,10uF,(2)
- added C19: 10uF, PCM_JLCPCB:C_CASE-A-3216-18(mm), symbol PCM_JLCPCB-Capacitors:CASE-A-3216-18(mm),10uF
- added C20, C21: 10uF, PCM_JLCPCB:C_0805, symbol PCM_JLCPCB-Capacitors:0805,10uF
- added C25: 10pF, PCM_JLCPCB:C_0402, symbol PCM_JLCPCB-Capacitors:0402,10pF
- added C28, C29: 22uF, PCM_JLCPCB:C_0805, symbol PCM_JLCPCB-Capacitors:0805,22uF
- added IC1: BQ24074RGTT, QFN50P300X300X100-17N-D, symbol Flight_computer:BQ24074RGTT
- added J1, J4: Conn_01x03_Socket, Connector_PinHeader_2.54mm:PinHeader_1x03_P2.54mm_Vertical, symbol Connector:Conn_01x03_Socket
- added J2: Conn_02x05_Odd_Even, Connector_PinHeader_1.27mm:PinHeader_2x05_P1.27mm_Vertical, symbol Connector_Generic:Conn_02x05_Odd_Even
- added J5: 104031-0811, 1040310811, symbol Flight_computer:104031-0811
- added J6: TB004-750-03GR, TB004-750-03GR, symbol Flight_computer:TB004-750-03GR
- added L3: L, Inductor_SMD:L_APV_APH0620, symbol Device:L
- added LED1, LED2: LTST-C190KGKT, LEDC1608X80N, symbol Flight_computer:LTST-C190KGKT
- added LS1: PS1240P02CT3, PS1240P02BT, symbol Flight_computer:PS1240P02CT3
- added PS1: TPS61033DRLR, SOTFL50P160X60-8N, symbol Flight_computer:TPS61033DRLR
- added R10, R22, R6, R9: 10kΩ, PCM_JLCPCB:R_0402, symbol PCM_JLCPCB-Resistors:0402,10kΩ
- added R11, R8: 1.5kΩ, PCM_JLCPCB:R_0402, symbol PCM_JLCPCB-Resistors:0402,1.5kΩ
- added R12, R13, R14, R15: 22Ω, PCM_JLCPCB:R_0402, symbol PCM_JLCPCB-Resistors:0402,22Ω
- added R16, R17, R20, R21: 1.1kΩ, PCM_JLCPCB:R_0603, symbol PCM_JLCPCB-Resistors:0603,1.1kΩ
- added R18: 750Ω, PCM_JLCPCB:R_0805, symbol PCM_JLCPCB-Resistors:0805,750Ω
- added R19: 49.9kΩ, PCM_JLCPCB:R_0402, symbol PCM_JLCPCB-Resistors:0402,49.9kΩ
Connections:
- net +3.3VP: now also C19.1, C6.1, J2.1 (Pin_1), J5.4 (VDD), LS1.2, R10.1, R11.1, R22.2, R8.1
- net +5V: now also C20.1, IC1.13 (IN), IC1.5 (EN2); no longer U1.3 (VIN)
- net Boot0: now also R6.2
- net D+: now also R8.2
- net GND: now also C15.2, C19.2, C20.2, C21.2, C25.2, C26.2, C27.2, C28.2, C29.2, C6.2, IC1.17 (EP), IC1.4 (~{CE}), IC1.6 (EN1), IC1.8 (VSS), J1.1 (Pin_1), J2.3 (Pin_3), J2.5 (Pin_5), J2.9 (Pin_9), J4.1 (Pin_1), J5.10, J5.11, J5.12, J5.13, J5.14, J5.6 (VSS), J5.9, J6.3, PS1.6 (GND), R16.2, R17.2, R18.2, R19.2, R6.1, R9.1; no longer U2.5 (CSB)
- net NRST: now also R15.2
- net SWCLK: now also R13.2
- net SWDIO: now also R12.2
- net SWO: now also R14.2
- net buzzer: now reaches U6.14 (PA4)
- net buzzer: now also LS1.1, R11.2
- net PG: now reaches U6.15 (PA5)
- net PG: now also PS1.4 (PG), R22.1
- net Boot1: now reaches U6.20 (PB2)
- net Boot1: now also R9.2
- net CD/DAT3: now reaches U6.25 (PB12)
- net CD/DAT3: now also J5.2 (CD/DAT3), R10.2
- net SPI2_SCK: now reaches U6.26 (PB13)
- net SPI2_SCK: now also J5.5 (CLK)
- net SPI2_MISO: now reaches U6.27 (PB14)
- net SPI2_MISO: now also J5.7 (DAT0)
- net SPI2_MOSI: now reaches U6.28 (PB15)
- net SPI2_MOSI: now also J5.3 (CMD)
- net S0: now reaches U6.45 (PB8)
- net S0: now also J1.3 (Pin_3)
- net S1: now reaches U6.46 (PB9)
- net S1: now also J4.3 (Pin_3)
- new net: J2.10 (Pin_10), R15.1
- new net: J2.2 (Pin_2), R12.1
- new net: J2.4 (Pin_4), R13.1
- new net: J2.6 (Pin_6), R14.1
- new net: LED2.2 (A), R20.1
- new net: LED1.2 (A), R21.1
- new net +5VD: C28.1, C29.1, J1.2 (Pin_2), J4.2 (Pin_2), PS1.8 (VOUT)
- new net BAT+: C21.1, IC1.2 (BAT_1), IC1.3 (BAT_2), J6.1
- new net CHG: IC1.9 (~{CHG}), LED2.1 (K)
- new net ILIM: IC1.12 (ILIM), R16.1
- new net ITERM: IC1.15 (ITERM), R17.1
- new net PGOOD: IC1.7 (~{PGOOD}), LED1.1 (K)
- new net R-ISET: IC1.16 (ISET), R18.1
- new net SW: L3.2, PS1.7 (SW)
- new net TMR: IC1.14 (TMR), R19.1
- new net TS: IC1.1 (TS), J6.2
- new net VDD: C15.1, C25.1, C26.1, C27.1, IC1.10 (OUT_1), IC1.11 (OUT_2), L3.1, PS1.1 (VIN), PS1.2 (EN), PS1.3 (MODE), PS1.5 (FB), R20.2, R21.2, U1.3 (VIN)
- no-connect marks 28 -> 24
Other:
- note added: "Battery and power supply"
- note added: "Buzzer"
- note added: "Decoupling capacitors"
- note added: "SD Card"
- note added: "STM Power regulator"
- note added: "Servo Power Supply"
- note added: "Servo connectors"
- note added: "USB Type-C interface"
- note removed: "C Type USB connection"
- note removed: "Decoupling Capacitors"
- note removed: "Power Regulator"
- company: (none) -> Yorha-7
- title: (none) -> Flight Computer
- moved on the sheet: C10, C13, C14, C17, C18, H1, H2, H3, H4, L2, R1, R2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
